File: KiCad/TL Kickoff T3.kicad_sch (KiCad schematic)
At the start: 0 parts

Commit message: Made a preliminary schematic, created helper functions for the distance sensor and installed the LED Strip component
Parts:
- added R1: 2K, symbol Device:R_Small_US
- added R2: 1K, symbol Device:R_Small_US
- added U1: ESP32-S3-DevKitC, PCM_Espressif:ESP32-S3-DevKitC, symbol PCM_Espressif:ESP32-S3-DevKitC
- added U2: (no value), symbol HC-SR04:HCSR04
- added U3: (no value), symbol NeoPixel LED Strip:NeoPixel_LED_Strip
Connections:
- new net: R2.1, U1.5 (GPIO5/ADC1_CH4)
- new net: U1.1 (3V3), U1.2 (3V3)
- new net +5V: U1.21 (5V), U2. (ECHO), U3. (DIN)
- new net ECHO: R1.1, R2.2, U2. (ECHO)
- new net GND: R1.2, U1.22 (GND), U1.23 (GND), U1.24 (GND), U1.44 (GND), U2. (ECHO), U3. (DIN)
- new net LEDOUT: U1.7 (GPIO7/ADC1_CH6), U3. (DIN)
- new net TRIG: U1.6 (GPIO6/ADC1_CH5), U2. (ECHO)
